Commit message: Fixed joint type

File: urdf/robot.urdf (robot description, URDF)
Before this commit: robot lab4, 5 links, 4 joints
Joints:
- joint base_laser_horiz_joint: type None -> fixed
- joint base_laser_vert_bottom_joint: type None -> fixed
- joint base_laser_vert_left_joint: type None -> fixed
- joint base_laser_vert_top_right_joint: type None -> fixed

Commit message: added left wheel

File: urdf/robot.urdf (robot description, URDF)
Before this commit: robot lab4, 5 links, 4 joints
Links:
- added link wheel_left; collision cylinder length=0.05 radius=0.2; visual cylinder length=0.05 radius=0.2
Joints:
- added joint base_wheel_left_joint: type fixed, parent base, child wheel_left, origin xyz=-0.10 0.4 0.0 rpy=-0.10 -0.4 0.0, limit lower=-2.2 upper=0.7 effort=30 velocity=1.0

Commit message: added rotation

File: urdf/robot.urdf (robot description, URDF)
Before this commit: robot lab4, 6 links, 5 joints
Joints:
- joint base_wheel_left_joint: origin xyz=-0.10 0.4 0.0 rpy=-0.10 -0.4 0.0 -> xyz=-0.10 0.4 0.0 rpy=-pi/2 0.0 0.0

Commit message: added readme and fixed typo in urdf

File: urdf/robot.urdf (robot description, URDF)
Before this commit: robot lab4, 6 links, 5 joints
Joints:
- removed joint base_laser_vert_left_joint
- added joint base_laser_vert_top_left_joint: type fixed, parent base, child laser_vert_top_left, origin xyz=0.2997 0.1531 1.8443 rpy=1.1780 0.6198 1.9560
