Commit message: Added xacro

File: urdf/robot.xacro (robot description, xacro)
@@ -1,4 +1,4 @@
 <?xml version="1.0"?>
-<robot name="lab4">
+<robot xmlns:xacro="http://www.ros.org/wiki/xacro" name="lab4">
     <link name="base">
         <visual>
@@ -98,24 +98,27 @@
         <child link="laser_horiz"/>
     </joint>
-    <link name="wheel_left">
-        <visual>
-            <geometry>
-                <cylinder radius="0.2" length="0.05" />
-            </geometry>
-            <material name="Red">
-                <color rgba="1.0 0 0 1.0"/>
-            </material>
-        </visual>
-        <collision>
-            <geometry>
-                <cylinder radius="0.2" length="0.05" />
-            </geometry>
-        </collision>
-    </link>
-    <joint name="base_wheel_left_joint" type="fixed">
-        <origin xyz="-0.10 0.4 0.0" rpy="-1.5708 0.0 0.0" />
-        <parent link="base"/>
-        <child link="wheel_left"/>
-        <limit effort="30" velocity="1.0" lower="-2.2" upper="0.7" />
-    </joint>
+    <xacro:macro name="xacro_name" params="suffix reflect">
+        <link name="wheel_${suffix}">
+            <visual>
+                <geometry>
+                    <cylinder radius="0.2" length="0.05" />
+                </geometry>
+                <material name="Red">
+                    <color rgba="1.0 0 0 1.0"/>
+                </material>
+            </visual>
+            <collision>
+                <geometry>
+                    <cylinder radius="0.2" length="0.05" />
+                </geometry>
+            </collision>
+        </link>
+        <joint name="base_wheel_${suffix}_joint" type="fixed">
+            <origin xyz="-0.10 0.4 0.0" rpy="-1.5708 0.0 0.0" />
+            <parent link="base"/>
+            <child link="wheel_${suffix}"/>
+            <limit effort="30" velocity="1.0" lower="-2.2" upper="0.7" />
+        </joint>
+    </xacro:macro>
+    <xacro:xacro_name suffix="left" reflect="1" />
 </robot>

Commit message: Center wheel

File: urdf/robot.xacro (robot description, xacro)
@@ -98,4 +98,25 @@
         <child link="laser_horiz"/>
     </joint>
+    <link name="wheel_center">
+        <visual>
+            <geometry>
+                <cylinder radius="0.15" length="0.05" />
+            </geometry>
+            <material name="Red">
+                <color rgba="1.0 0 0 1.0"/>
+            </material>
+        </visual>
+        <collision>
+            <geometry>
+                <cylinder radius="0.15" length="0.05" />
+            </geometry>
+        </collision>
+    </link>
+    <joint name="base_wheel_center_joint" type="fixed">
+        <origin xyz="0.1 0.0 0.0" rpy="-1.5708 0.0 0.0" />
+        <parent link="base"/>
+        <child link="wheel_center"/>
+        <limit effort="30" velocity="1.0" lower="-2.2" upper="0.7" />
+    </joint>
     <xacro:macro name="xacro_name" params="suffix reflect">
         <link name="wheel_${suffix}">
@@ -115,5 +136,5 @@
         </link>
         <joint name="base_wheel_${suffix}_joint" type="fixed">
-            <origin xyz="-0.10 0.4 0.0" rpy="-1.5708 0.0 0.0" />
+            <origin xyz="-0.10 ${reflect * 0.4} 0.0" rpy="-1.5708 0.0 0.0" />
             <parent link="base"/>
             <child link="wheel_${suffix}"/>
@@ -122,3 +143,4 @@
     </xacro:macro>
     <xacro:xacro_name suffix="left" reflect="1" />
+    <xacro:xacro_name suffix="right" reflect="-1" />
 </robot>

Commit message: Continuous joints

File: urdf/robot.xacro (robot description, xacro)
@@ -113,9 +113,9 @@
         </collision>
     </link>
-    <joint name="base_wheel_center_joint" type="fixed">
+    <joint name="base_wheel_center_joint" type="continuous">
         <origin xyz="0.1 0.0 0.0" rpy="-1.5708 0.0 0.0" />
         <parent link="base"/>
         <child link="wheel_center"/>
-        <limit effort="30" velocity="1.0" lower="-2.2" upper="0.7" />
+        <limit effort="30" velocity="1.0"/>
     </joint>
     <xacro:macro name="xacro_name" params="suffix reflect">
@@ -135,9 +135,9 @@
             </collision>
         </link>
-        <joint name="base_wheel_${suffix}_joint" type="fixed">
+        <joint name="base_wheel_${suffix}_joint" type="continuous">
             <origin xyz="-0.10 ${reflect * 0.4} 0.0" rpy="-1.5708 0.0 0.0" />
             <parent link="base"/>
             <child link="wheel_${suffix}"/>
-            <limit effort="30" velocity="1.0" lower="-2.2" upper="0.7" />
+            <limit effort="30" velocity="1.0"/>
         </joint>
     </xacro:macro>

Commit message: change axis

File: urdf/robot.xacro (robot description, xacro)
@@ -117,4 +117,5 @@
         <parent link="base"/>
         <child link="wheel_center"/>
+        <axis xyz="0 0 1"/>
         <limit effort="30" velocity="1.0"/>
     </joint>
@@ -139,4 +140,5 @@
             <parent link="base"/>
             <child link="wheel_${suffix}"/>
+            <axis xyz="0 0 1"/>
             <limit effort="30" velocity="1.0"/>
         </joint>

Commit message: Added Velodyne

File: urdf/robot.xacro (robot description, xacro)
@@ -3,4 +3,10 @@
     <xacro:include filename="$(find gazebo_plugins)/test/multi_robot_scenario/xacro/laser/hokuyo.xacro"/>
     <!--<xacro:include filename="$(find velodyne_description)/urdf/VLP-16.urdf.xacro"/>-->
+    <!--
+        This package was not installed on the jennings machines so I downloaded the xacro.
+        Should be this
+        <xacro:include filename="$(find velodyne_description)/urdf/VLP-16.urdf.xacro"/>
+    -->
+    <xacro:include filename="$(find urdf_lab)/urdf/VLP-16.urdf.xacro"/>
     <link name="base">
         <visual>
@@ -112,5 +118,7 @@
     </link>
     -->
-    <xacro:laser name="laser_horiz" parent="base" xyz="0.2325 0.0001 1.9201" rpy="-0.0012068 0.114646 -0.0015308" meshes="package://gazebo_plugins/test/multi_robot_scenario/meshes/laser" />
+    <VLP-16 parent="base" name="laser_horiz" topic="laser_horiz/packets" hz="10" samples="440" gpu="false">
+        <origin xyz="0.2325416305773505 -0.0001380069427607134 1.920122926231907" rpy="-0.0012068 0.114646 -0.0015308" />
+    </VLP-16>
     <!--
     <joint name="base_laser_horiz_joint" type="fixed">

Commit message: Updated xacro

File: urdf/robot.xacro (robot description, xacro)
@@ -2,5 +2,4 @@
 <robot xmlns:xacro="http://www.ros.org/wiki/xacro" name="lab4">
     <xacro:include filename="$(find gazebo_plugins)/test/multi_robot_scenario/xacro/laser/hokuyo.xacro"/>
-    <!--<xacro:include filename="$(find velodyne_description)/urdf/VLP-16.urdf.xacro"/>-->
     <xacro:include filename="$(find velodyne_description)/urdf/VLP-16.urdf.xacro"/>
     <link name="base">
@@ -21,4 +20,52 @@
         </collision>
     </link>
+    <link name="wheel_center">
+        <visual>
+            <geometry>
+                <cylinder radius="0.15" length="0.05" />
+            </geometry>
+            <material name="Red">
+                <color rgba="1.0 0 0 1.0"/>
+            </material>
+        </visual>
+        <collision>
+            <geometry>
+                <cylinder radius="0.15" length="0.05" />
+            </geometry>
+        </collision>
+    </link>
+    <joint name="base_wheel_center_joint" type="continuous">
+        <origin xyz="0.1 0.0 0.0" rpy="-1.5708 0.0 0.0" />
+        <parent link="base"/>
+        <child link="wheel_center"/>
+        <axis xyz="0 0 1"/>
+        <limit effort="30" velocity="1.0"/>
+    </joint>
+    <xacro:macro name="xacro_name" params="suffix reflect">
+        <link name="wheel_${suffix}">
+            <visual>
+                <geometry>
+                    <cylinder radius="0.2" length="0.05" />
+                </geometry>
+                <material name="Red">
+                    <color rgba="1.0 0 0 1.0"/>
+                </material>
+            </visual>
+            <collision>
+                <geometry>
+                    <cylinder radius="0.2" length="0.05" />
+                </geometry>
+            </collision>
+        </link>
+        <joint name="base_wheel_${suffix}_joint" type="continuous">
+            <origin xyz="-0.10 ${reflect * 0.4} 0.0" rpy="-1.5708 0.0 0.0" />
+            <parent link="base"/>
+            <child link="wheel_${suffix}"/>
+            <axis xyz="0 0 1"/>
+            <limit effort="30" velocity="1.0"/>
+        </joint>
+    </xacro:macro>
+    <xacro:xacro_name suffix="left" reflect="1" />
+    <xacro:xacro_name suffix="right" reflect="-1" />
     <!--
     <link name="laser_vert_bottom">
@@ -38,5 +85,4 @@
     </link>
     -->
-    <!--<xacro:laser name="laser_vert_test" parent="base" xyz="0.2997 1.5 1.8443" rpy="1.1780 0.6198 1.9560" meshes="package://gazebo_plugins/test/multi_robot_scenario/meshes/laser" />-->
     <xacro:laser name="laser_vert_bottom" parent="base" xyz="0.3157894464801903 -0.002068548615034871 0.5099999434059285" rpy="3.1354753 -1.3045001 0.0024658" meshes="package://gazebo_plugins/test/multi_robot_scenario/meshes/laser" />
     <!--
@@ -124,51 +170,3 @@
     </joint>
     -->
-    <link name="wheel_center">
-        <visual>
-            <geometry>
-                <cylinder radius="0.15" length="0.05" />
-            </geometry>
-            <material name="Red">
-                <color rgba="1.0 0 0 1.0"/>
-            </material>
-        </visual>
-        <collision>
-            <geometry>
-                <cylinder radius="0.15" length="0.05" />
-            </geometry>
-        </collision>
-    </link>
-    <joint name="base_wheel_center_joint" type="continuous">
-        <origin xyz="0.1 0.0 0.0" rpy="-1.5708 0.0 0.0" />
-        <parent link="base"/>
-        <child link="wheel_center"/>
-        <axis xyz="0 0 1"/>
-        <limit effort="30" velocity="1.0"/>
-    </joint>
-    <xacro:macro name="xacro_name" params="suffix reflect">
-        <link name="wheel_${suffix}">
-            <visual>
-                <geometry>
-                    <cylinder radius="0.2" length="0.05" />
-                </geometry>
-                <material name="Red">
-                    <color rgba="1.0 0 0 1.0"/>
-                </material>
-            </visual>
-            <collision>
-                <geometry>
-                    <cylinder radius="0.2" length="0.05" />
-                </geometry>
-            </collision>
-        </link>
-        <joint name="base_wheel_${suffix}_joint" type="continuous">
-            <origin xyz="-0.10 ${reflect * 0.4} 0.0" rpy="-1.5708 0.0 0.0" />
-            <parent link="base"/>
-            <child link="wheel_${suffix}"/>
-            <axis xyz="0 0 1"/>
-            <limit effort="30" velocity="1.0"/>
-        </joint>
-    </xacro:macro>
-    <xacro:xacro_name suffix="left" reflect="1" />
-    <xacro:xacro_name suffix="right" reflect="-1" />
 </robot>
