Commit message: Revert "Copied another file"
This reverts commit a5ade66c47e408554bb7399f9956ab17cb1fa504.

File: urdf/robot.xacro (robot description, xacro)
@@ -1,160 +1,172 @@
 <?xml version="1.0"?>
-<robot xmlns:xacro="http://www.ros.org/wiki/xacro" name="robot">
-<!--INCLUDING OTHER FILES-->
-<!-- Include the XACRO file that defines a Hokuyo LIDAR. -->
-<xacro:include filename="$(find gazebo_plugins)/test/multi_robot_scenario/xacro/laser/hokuyo.xacro" />
-<!-- Include the XACRO file that defines a Hokuyo LIDAR. -->
-  <xacro:include filename="$(find velodyne_description)/urdf/VLP-16.urdf.xacro"/>
-<!--  position wrt parent == origin; orientation == rpy  -->
-<!--  units are in meters  -->
-<!--  if you do not put in an origin, it defaults to the COM  -->
- <!--LINKS-->
-        <link name = "base">
-                <visual>
-                        <origin xyz="0 0 0.99" rpy="0 0 0"/>
-	                <geometry>
-	                        <box size="0.94 0.78 1.98" />
-	                </geometry>
- 	        </visual>
-	        <collision>
-                        <origin xyz="0 0 0.99" rpy="0 0 0"/>
-	                <geometry>
-	                        <box size="0.94 0.78 1.98" />
-	                </geometry>
-	        </collision>
+<robot xmlns:xacro="http://www.ros.org/wiki/xacro" name="lab4">
+    <xacro:include filename="$(find gazebo_plugins)/test/multi_robot_scenario/xacro/laser/hokuyo.xacro"/>
+    <xacro:include filename="$(find velodyne_description)/urdf/VLP-16.urdf.xacro"/>
+    <link name="base">
+        <visual>
+            <origin xyz="0 0 0.99" rpy="0 0 0" />
+            <geometry>
+                <box size="0.94 0.78 1.98" />
+            </geometry>
+            <material name="Cyan">
+                <color rgba="0 1.0 1.0 0.5"/>
+            </material>
+        </visual>
+        <collision>
+            <origin xyz="0 0 0.99" rpy="0 0 0"/>
+            <geometry>
+                <box size="0.94 0.78 1.98" />
+            </geometry>
+        </collision>
+    </link>
+    <link name="wheel_center">
+        <visual>
+            <geometry>
+                <cylinder radius="0.15" length="0.05" />
+            </geometry>
+            <material name="Red">
+                <color rgba="1.0 0 0 1.0"/>
+            </material>
+        </visual>
+        <collision>
+            <geometry>
+                <cylinder radius="0.15" length="0.05" />
+            </geometry>
+        </collision>
+    </link>
+    <joint name="base_wheel_center_joint" type="continuous">
+        <origin xyz="0.1 0.0 0.0" rpy="-1.5708 0.0 0.0" />
+        <parent link="base"/>
+        <child link="wheel_center"/>
+        <axis xyz="0 0 1"/>
+        <limit effort="30" velocity="1.0"/>
+    </joint>
+    <xacro:macro name="xacro_name" params="suffix reflect">
+        <link name="wheel_${suffix}">
+            <visual>
+                <geometry>
+                    <cylinder radius="0.2" length="0.05" />
+                </geometry>
+                <material name="Red">
+                    <color rgba="1.0 0 0 1.0"/>
+                </material>
+            </visual>
+            <collision>
+                <geometry>
+                    <cylinder radius="0.2" length="0.05" />
+                </geometry>
+            </collision>
         </link>
-<!--
-        <link name = "laser_vert_bottom">
-	        <visual>
-	                <geometry>
-	                        <box size="0.062 0.062 0.087" />
-	                </geometry>
- 	        </visual>
-	        <collision>
-	                <geometry>
-	                        <box size="0.062 0.062 0.087" />
-	                </geometry>
-	        </collision>
-        </link>
-        <link name = "laser_vert_top_right">
-	        <visual>
-	                <geometry>
-	                        <box size="0.062 0.062 0.087" />
-	                </geometry>
- 	        </visual>
-	        <collision>
-	                <geometry>
-	                        <box size="0.062 0.062 0.087" />
-	                </geometry>
-	        </collision>
-        </link>
-        <link name = "laser_vert_top_left">
-	        <visual>
-	                <geometry>
-	                        <box size="0.062 0.062 0.087" />
-	                </geometry>
- 	        </visual>
-	        <collision>
-	                <geometry>
-	                        <box size="0.062 0.062 0.087" />
-	                </geometry>
-	        </collision>
-        </link>
-        <link name = "laser_horiz">
-	        <visual>
-	                <geometry>
-	                        <cylinder radius="0.052" length="0.072"/>
-	                </geometry>
- 	                </visual>
-	        <collision>
-	                <geometry>
-	                        <cylinder radius="0.052" length="0.072"/>
-	                </geometry>
-	        </collision>
-        </link>
- -->
- <!--WHEELS-->
-<xacro:macro name="xacro_name" params="suffix reflect">
-        <link name = "wheel_${suffix}">
-	        <visual>
-	                <geometry>
-	                        <cylinder radius="0.2" length="0.05"/>
-	                </geometry>
- 	                </visual>
-	        <collision>
-	                <geometry>
-	                        <cylinder radius="0.2" length="0.05"/>
-	                </geometry>
-	        </collision>
-        </link>
-        <joint name="wheel_${suffix}_joint" type="continuous">
-                <origin xyz="-0.10 ${reflect*0.4} 0.0" rpy="-${pi/2} 0 0"/>
-                <parent link="base"/>
-                <child link="wheel_${suffix}"/>
-                <axis xyz = "0 0 1"/>
+        <joint name="base_wheel_${suffix}_joint" type="continuous">
+            <origin xyz="-0.10 ${reflect * 0.4} 0.0" rpy="-1.5708 0.0 0.0" />
+            <parent link="base"/>
+            <child link="wheel_${suffix}"/>
+            <axis xyz="0 0 1"/>
+            <limit effort="30" velocity="1.0"/>
         </joint>
-</xacro:macro>
-<xacro:xacro_name suffix="left" reflect="1" />
-<xacro:xacro_name suffix="right" reflect="-1" />
-        <link name = "wheel_center">
-	        <visual>
-	                <!--<origin xyz="0 0 0" rpy="-0.0012068 0.114646 -0.0015308"/>-->
-	                <geometry>
-	                        <cylinder radius="0.15" length="0.05"/>
-	                </geometry>
- 	                </visual>
-	        <collision>
-	                <!--<origin xyz="0 0 0" rpy="-0.0012068 0.114646 -0.0015308"/> -->
-	                <geometry>
-	                        <cylinder radius="0.15" length="0.05"/>
-	                </geometry>
-	        </collision>
-        </link>
-        <joint name="wheel_center_joint" type="continuous">
-                <origin xyz="0.10 0 0" rpy="-${pi/2} 0 0"/>
-                <parent link="base"/>
-                <child link="wheel_center"/>
-                <axis xyz = "0 0 1"/>
-        </joint>
- <!--JOINTS-->
- <!-- Include the XACRO file that defines a Hokuyo LIDAR. -->
- <!--        <joint name="base_laser_vert_bottom_joint" type="fixed">
-                <origin xyz="0.3158 -0.0021 0.5100" rpy="3.1355 -1.3045 0.0025"/>
-                <parent link="base"/>
-                <child link="laser_vert_bottom"/>
-        </joint>
--->
-        <xacro:laser name="laser_vert_bottom" parent="base" xyz="0.3157894464801903
-        -0.002068548615034871 0.5099999434059285" rpy="3.1354753 -1.3045001 0.0024658"
-        meshes="package://gazebo_plugins/test/multi_robot_scenario/meshes/laser" />
- <!--
-        <joint name="base_laser_vert_top_right_joint" type="fixed">
-                <origin xyz="0.2978 -0.1450 1.8451" rpy="-1.1760 0.6313 1.9377"/>
-                <parent link="base"/>
-                <child link="laser_vert_top_right"/>
-        </joint>
--->
-        <xacro:laser name="laser_vert_top_right" parent="base" xyz="0.2978 -0.1450 1.8451" rpy="-1.1760 0.6313 1.9377"
-        meshes="package://gazebo_plugins/test/multi_robot_scenario/meshes/laser" />
-<!--
-        <joint name="base_laser_vert_top_left_joint" type="fixed">
-                <origin xyz="0.2997 0.1531 1.8443" rpy="1.1780 0.6198 1.9560"/>
-                <parent link="base"/>
-                <child link="laser_vert_top_left"/>
-        </joint>
--->
-         <xacro:laser name="laser_vert_top_left" parent="base" xyz="0.2997 0.1531 1.8443" rpy="1.1780 0.6198     1.9560"
-        meshes="package://gazebo_plugins/test/multi_robot_scenario/meshes/laser" />
-<!--        <joint name="base_laser_horiz_joint" type="fixed">
-                <origin xyz="0.2325 0.0001 1.9201" rpy="-0.0012068 0.114646 -0.0015308"/>
-                <parent link="base"/>
-                <child link="laser_horiz"/>
-        </joint>
--->
-<!-- Invoke the macro to define the Hokuyo LIDAR. -->
-  <VLP-16 parent="base" name="laser_horiz" topic="laser_horiz/packets" hz="10"
-samples="440" gpu="false">
-       <origin xyz="0.2325416305773505 -0.0001380069427607134 1.920122926231907"
-rpy="-0.0012068 0.114646 -0.0015308" />
-  </VLP-16>
+    </xacro:macro>
+    <xacro:xacro_name suffix="left" reflect="1" />
+    <xacro:xacro_name suffix="right" reflect="-1" />
+    <!--
+    <link name="laser_vert_bottom">
+        <visual>
+            <geometry>
+                <box size="0.0062 0.0062 0.0087" />
+            </geometry>
+            <material name="Red">
+                <color rgba="1.0 0 0 1.0"/>
+            </material>
+        </visual>
+        <collision>
+            <geometry>
+                <box size="0.0062 0.0062 0.0087" />
+            </geometry>
+        </collision>
+    </link>
+    -->
+    <xacro:laser name="laser_vert_bottom" parent="base" xyz="0.3157894464801903 -0.002068548615034871 0.5099999434059285" rpy="3.1354753 -1.3045001 0.0024658" meshes="package://gazebo_plugins/test/multi_robot_scenario/meshes/laser" />
+    <!--
+    <joint name="base_laser_vert_bottom_joint" type="fixed">
+        <origin xyz="0.3158 -0.0021 0.5100" rpy="3.1355 -1.3045 0.0025" />
+        <parent link="base"/>
+        <child link="laser_vert_bottom"/>
+    </joint>
+    -->
+    <!--
+    <link name="laser_vert_top_right">
+        <visual>
+            <geometry>
+                <box size="0.0062 0.0062 0.0087" />
+            </geometry>
+            <material name="Red">
+                <color rgba="1.0 0 0 1.0"/>
+            </material>
+        </visual>
+        <collision>
+            <geometry>
+                <box size="0.0062 0.0062 0.0087" />
+            </geometry>
+        </collision>
+    </link>
+    -->
+    <xacro:laser name="laser_vert_top_right" parent="base" xyz="0.2978 -0.1450 1.8451" rpy="-1.1760 0.6313 -1.9377" meshes="package://gazebo_plugins/test/multi_robot_scenario/meshes/laser" />
+    <!--
+    <joint name="base_laser_vert_top_right_joint" type="fixed">
+        <origin xyz="0.2978 -0.1450 1.8451" rpy="-1.1760 0.6313 -1.9377" />
+        <parent link="base"/>
+        <child link="laser_vert_top_right"/>
+    </joint>
+    -->
+    <!--
+    <link name="laser_vert_top_left">
+        <visual>
+            <geometry>
+                <box size="0.0062 0.0062 0.0087" />
+            </geometry>
+            <material name="Red">
+                <color rgba="1.0 0 0 1.0"/>
+            </material>
+        </visual>
+        <collision>
+            <geometry>
+                <box size="0.0062 0.0062 0.0087" />
+            </geometry>
+        </collision>
+    </link>
+    -->
+    <xacro:laser name="laser_vert_top_left" parent="base" xyz="0.2997 0.1531 1.8443" rpy="1.1780 0.6198 1.9560" meshes="package://gazebo_plugins/test/multi_robot_scenario/meshes/laser" />
+    <!--
+    <joint name="base_laser_vert_left_joint" type="fixed">
+        <origin xyz="0.2997 0.1531 1.8443" rpy="1.1780 0.6198 1.9560" />
+        <parent link="base"/>
+        <child link="laser_vert_top_left"/>
+    </joint>
+    -->
+    <!--
+    <link name="laser_horiz">
+        <visual>
+            <geometry>
+                <cylinder radius="0.0052" length="0.0072" />
+            </geometry>
+            <material name="Red">
+                <color rgba="1.0 0 0 1.0"/>
+            </material>
+        </visual>
+        <collision>
+            <geometry>
+                <cylinder radius="0.0052" length="0.0072" />
+            </geometry>
+        </collision>
+    </link>
+    -->
+    <VLP-16 parent="base" name="laser_horiz" topic="laser_horiz/packets" hz="10" samples="440" gpu="false">
+        <origin xyz="0.2325416305773505 -0.0001380069427607134 1.920122926231907" rpy="-0.0012068 0.114646 -0.0015308" />
+    </VLP-16>
+    <!--
+    <joint name="base_laser_horiz_joint" type="fixed">
+        <origin xyz="0.2325 0.0001 1.9201" rpy="-0.0012068 0.114646 -0.0015308" />
+        <parent link="base"/>
+        <child link="laser_horiz"/>
+    </joint>
+    -->
 </robot>

Commit message: Revert "Updated xacro"
This reverts commit bd7ce1c460376cfd1de7d413c87d009e16879795.

File: urdf/robot.xacro (robot description, xacro)
@@ -2,4 +2,5 @@
 <robot xmlns:xacro="http://www.ros.org/wiki/xacro" name="lab4">
     <xacro:include filename="$(find gazebo_plugins)/test/multi_robot_scenario/xacro/laser/hokuyo.xacro"/>
+    <!--<xacro:include filename="$(find velodyne_description)/urdf/VLP-16.urdf.xacro"/>-->
     <xacro:include filename="$(find velodyne_description)/urdf/VLP-16.urdf.xacro"/>
     <link name="base">
@@ -20,52 +21,4 @@
         </collision>
     </link>
-    <link name="wheel_center">
-        <visual>
-            <geometry>
-                <cylinder radius="0.15" length="0.05" />
-            </geometry>
-            <material name="Red">
-                <color rgba="1.0 0 0 1.0"/>
-            </material>
-        </visual>
-        <collision>
-            <geometry>
-                <cylinder radius="0.15" length="0.05" />
-            </geometry>
-        </collision>
-    </link>
-    <joint name="base_wheel_center_joint" type="continuous">
-        <origin xyz="0.1 0.0 0.0" rpy="-1.5708 0.0 0.0" />
-        <parent link="base"/>
-        <child link="wheel_center"/>
-        <axis xyz="0 0 1"/>
-        <limit effort="30" velocity="1.0"/>
-    </joint>
-    <xacro:macro name="xacro_name" params="suffix reflect">
-        <link name="wheel_${suffix}">
-            <visual>
-                <geometry>
-                    <cylinder radius="0.2" length="0.05" />
-                </geometry>
-                <material name="Red">
-                    <color rgba="1.0 0 0 1.0"/>
-                </material>
-            </visual>
-            <collision>
-                <geometry>
-                    <cylinder radius="0.2" length="0.05" />
-                </geometry>
-            </collision>
-        </link>
-        <joint name="base_wheel_${suffix}_joint" type="continuous">
-            <origin xyz="-0.10 ${reflect * 0.4} 0.0" rpy="-1.5708 0.0 0.0" />
-            <parent link="base"/>
-            <child link="wheel_${suffix}"/>
-            <axis xyz="0 0 1"/>
-            <limit effort="30" velocity="1.0"/>
-        </joint>
-    </xacro:macro>
-    <xacro:xacro_name suffix="left" reflect="1" />
-    <xacro:xacro_name suffix="right" reflect="-1" />
     <!--
     <link name="laser_vert_bottom">
@@ -85,4 +38,5 @@
     </link>
     -->
+    <!--<xacro:laser name="laser_vert_test" parent="base" xyz="0.2997 1.5 1.8443" rpy="1.1780 0.6198 1.9560" meshes="package://gazebo_plugins/test/multi_robot_scenario/meshes/laser" />-->
     <xacro:laser name="laser_vert_bottom" parent="base" xyz="0.3157894464801903 -0.002068548615034871 0.5099999434059285" rpy="3.1354753 -1.3045001 0.0024658" meshes="package://gazebo_plugins/test/multi_robot_scenario/meshes/laser" />
     <!--
@@ -170,3 +124,51 @@
     </joint>
     -->
+    <link name="wheel_center">
+        <visual>
+            <geometry>
+                <cylinder radius="0.15" length="0.05" />
+            </geometry>
+            <material name="Red">
+                <color rgba="1.0 0 0 1.0"/>
+            </material>
+        </visual>
+        <collision>
+            <geometry>
+                <cylinder radius="0.15" length="0.05" />
+            </geometry>
+        </collision>
+    </link>
+    <joint name="base_wheel_center_joint" type="continuous">
+        <origin xyz="0.1 0.0 0.0" rpy="-1.5708 0.0 0.0" />
+        <parent link="base"/>
+        <child link="wheel_center"/>
+        <axis xyz="0 0 1"/>
+        <limit effort="30" velocity="1.0"/>
+    </joint>
+    <xacro:macro name="xacro_name" params="suffix reflect">
+        <link name="wheel_${suffix}">
+            <visual>
+                <geometry>
+                    <cylinder radius="0.2" length="0.05" />
+                </geometry>
+                <material name="Red">
+                    <color rgba="1.0 0 0 1.0"/>
+                </material>
+            </visual>
+            <collision>
+                <geometry>
+                    <cylinder radius="0.2" length="0.05" />
+                </geometry>
+            </collision>
+        </link>
+        <joint name="base_wheel_${suffix}_joint" type="continuous">
+            <origin xyz="-0.10 ${reflect * 0.4} 0.0" rpy="-1.5708 0.0 0.0" />
+            <parent link="base"/>
+            <child link="wheel_${suffix}"/>
+            <axis xyz="0 0 1"/>
+            <limit effort="30" velocity="1.0"/>
+        </joint>
+    </xacro:macro>
+    <xacro:xacro_name suffix="left" reflect="1" />
+    <xacro:xacro_name suffix="right" reflect="-1" />
 </robot>
